Commit message: feat: Funciona ya el slam karto

File: urdf/mecanum_base.urdf (robot description, URDF)
Before this commit: robot mecanum_base, 2 links, 1 joints
Links:
- removed link scan
- added link laser
Joints:
- removed joint base_scan
- added joint base_laser_joint: type fixed, parent base_link, child laser, origin xyz=0.06 0.00 0.08 rpy=0 0 0
